File: KiCad Files/RFID_NFC_TAG_9x6.kicad_sch (KiCad schematic)
At the start: 4 parts, among them U1 SL2S2602FTBX

Commit message: Tag Updates After Testing
Parts:
- C1: value 43pF -> 51pF
- U1: footprint XSON3_SL2S2602_NXP -> NFC Tag Chip:XSON3_SL2S2602_NXP
Changed lines of the file:
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@@
 	(paper "A4")
-	(junction
-		(at 170.18 60.96)
-		(diameter 0)
-		(color 0 0 0 0)
-	)
 	(junction
 		(at 170.18 73.66)
@@
 	)
 	(junction
-		(at 170.18 99.06)
+		(at 170.18 58.42)
 		(diameter 0)
 		(color 0 0 0 0)
@@
 	(wire
 		(pts
-			(xy 170.18 60.96) (xy 170.18 73.66)
-		)
-		(stroke
-			(width 0)
-			(type default)
-		)
-	)
-	(wire
-		(pts
-			(xy 170.18 99.06) (xy 170.18 100.965)
-		)
-		(stroke
-			(width 0)
-			(type default)
-		)
-	)
-	(wire
-		(pts
 			(xy 182.88 83.82) (xy 190.5 83.82)
 		)
@@
 	(wire
 		(pts
-			(xy 170.18 58.42) (xy 170.18 60.96)
+			(xy 170.18 58.42) (xy 170.18 73.66)
 		)
 		(stroke
@@
 	(wire
 		(pts
-			(xy 170.18 60.96) (xy 172.72 60.96)
+			(xy 170.18 58.42) (xy 172.72 58.42)
 		)
 		(stroke
@@
 	(wire
 		(pts
-			(xy 132.08 100.965) (xy 132.08 99.06)
-		)
-		(stroke
-			(width 0)
-			(type default)
-		)
-	)
-	(wire
-		(pts
 			(xy 170.18 83.82) (xy 170.18 99.06)
 		)
@@
 	(wire
 		(pts
-			(xy 132.08 100.965) (xy 170.18 100.965)
+			(xy 132.08 99.06) (xy 170.18 99.06)
 		)
 		(stroke
@@
 		(pts
 			(xy 170.18 83.82) (xy 177.8 83.82)
-		)
-		(stroke
-			(width 0)
-			(type default)
-		)
-	)
-	(wire
-		(pts
-			(xy 170.18 99.06) (xy 173.355 99.06)
 		)
 		(stroke
@@
 	(global_label "ANT_LB"
 		(shape passive)
-		(at 172.72 99.06 0)
+		(at 170.18 99.06 0)
 		(fields_autoplaced yes)
 		(effects
@@
 		)
 		(property "Intersheetrefs" "${INTERSHEET_REFS}"
-			(at 181.2463 99.06 0)
+			(at 178.7063 99.06 0)
 			(effects
 				(font
@@
 	(global_label "ANT_LA"
 		(shape passive)
-		(at 172.72 60.96 0)
+		(at 172.72 58.42 0)
 		(fields_autoplaced yes)
 		(effects
@@
 		)
 		(property "Intersheetrefs" "${INTERSHEET_REFS}"
-			(at 181.0649 60.96 0)
+			(at 181.0649 58.42 0)
 			(effects
 				(font
@@
 			)
 		)
-		(property "Value" "43pF"
+		(property "Value" "51pF"
 			(at 173.99 80.0099 0)
 			(effects
@@
 			)
 		)
-		(property "Footprint" "XSON3_SL2S2602_NXP"
+		(property "Footprint" "NFC Tag Chip:XSON3_SL2S2602_NXP"
 			(at 132.08 99.06 0)
 			(effects
